Commit message: simulasi gazebo dengan lapangan robocon dan menggunakan slam_toolbox sudah bisa

File: description/diff_drive_description.urdf (robot description, URDF)
Before this commit: robot sam_bot, 7 links, 6 joints
Joints:
- joint lidar_joint: origin xyz=0 0 0.12 rpy=0 0 0 -> xyz=0.265 0 -0.1 rpy=0 0 0
